File: kicadproject/kyanit.kicad_pcb (KiCad board)
At the start: 2 copper layers, 79.8 x 69.1 mm, 32 parts, among them J1 TBUS, J2 PWR, J4 USB Micro-B, J5 Prog Conn, SW1 SW_Push, SW2 SW_Push, U1 USBLC6-2SC6, U2 HT7233, U3 CH330, U4 ESP-12F

Commit message: feat: rename gpio nets, add pinout to silkscreen
Parts:
- F1: value 200mA -> 500mA
- F2: value 1A -> 500mA
Connections:
- net CS0 renamed CS
- net D0 renamed GPIO16
- net D1 renamed GPIO5
- net D2 renamed GPIO9
- net D3 renamed GPIO10
- net D4 renamed GPIO12
- net D5 renamed GPIO13
- net ESP_nRTS renamed ESP_nRST
Other:
- board text added: "10"
- board text added: "12"
- board text added: "13"
- board text added: "16"
- board text added: "5"
- board text added: "5V"
- board text added: "9"
- board text added: "GND"
- board text added: "cs"
- board text added: "miso"
- board text added: "mosi"
- board text added: "sclk"
